Commit message: feat(yam): reorient FT-sensor frame + push sensor/gripper outward
g1_29dof_yam.urdf, both hands:
- Rotate the ft_sensor link frame rpy="0 -pi/2 pi" so the sensor axes
  follow the real FT convention (sensor +z -> wrist +x forward, +x -> +z
  up, +y -> -y). Child origins carry compensating transforms so the
  gripper's world pose is byte-for-byte unchanged (verified 4e-10 drift).
- Move the FT sensor +1 cm outward along wrist +x (0.072 -> 0.082).
- Add +2 cm gripper-vs-sensor standoff (palm local z 0.0095 -> 0.0295),
  so the gripper base sits at wrist +x 0.1115 (+3 cm net from the wrist).

Co-Authored-By: Claude Opus 4.8 (1M context) <noreply@anthropic.com>

File: src/holosoma/holosoma/data/robots/g1/g1_29dof_yam.urdf (robot description, URDF)
Before this commit: robot g1, 48 links, 47 joints
Joints:
- joint left_ft_sensor_joint: origin xyz=0.072 0 0 rpy=0 0 0 -> xyz=0.082 0 0 rpy=0 -1.570796327 3.141592654
- joint left_hand_palm_joint: origin xyz=0.0095 0.003 0 rpy=0 0 0 -> xyz=0 -0.003 0.0295 rpy=0 -1.570796327 3.141592654
- joint right_ft_sensor_joint: origin xyz=0.072 0 0 rpy=0 0 0 -> xyz=0.082 0 0 rpy=0 -1.570796327 3.141592654
- joint right_hand_palm_joint: origin xyz=0.0095 -0.003 0 rpy=0 0 0 -> xyz=0 0.003 0.0295 rpy=0 -1.570796327 3.141592654

Commit message: feat(g1-yam): update FT sensor + YAM gripper masses to real hardware
FT sensor link 0.1 -> 0.25 kg (isotropic inertia 3e-5 -> 7.5e-5), YAM gripper
total 0.695 -> 1.25 kg (rubber_hand base 0.553219 -> 1.107992, inertia scaled
x2.0028; two fingers unchanged). Both hands, symmetric. Distal mass on the
wrist F/T sensor is now ~1.5 kg, matching the real Bota puck + i2rt linear_4310.

Rationale for the hybrid position-force controller: the distal mass sets the
inertial pseudo-force (m*a) the wrist F/T sensor reads under acceleration even
with no contact, so it must match hardware for sim-to-real.

NOTE: this is a mass-only + proportional-inertia-scale edit. Because the added
mass is non-uniform (FT puck vs gripper base), the fused-body COM in the
hand-authored MJCF (g1_29dof_yam.xml) should be regenerated via
collapse_fixed_joints rather than hand-scaled -- tracked separately.

Co-Authored-By: Claude Opus 4.8 (1M context) <noreply@anthropic.com>

File: src/holosoma/holosoma/data/robots/g1/g1_29dof_yam.urdf (robot description, URDF)
Before this commit: robot g1, 48 links, 47 joints
Links:
- link left_ft_sensor_link: mass 0.1 -> 0.25
- link left_rubber_hand: mass 0.553219 -> 1.107992
- link right_ft_sensor_link: mass 0.1 -> 0.25
- link right_rubber_hand: mass 0.553219 -> 1.107992

Commit message: fix(g1-yam): gripper standoff 0.0295->0.0565 m so TCP reaches wrist +x 0.242
Re-parented gripper's palm-vs-FT-sensor standoff was 0.0295 m, putting the gripper
base at wrist +x 0.1115 and the fingertips short of the calibrated grasp point.
Bump the standoff to 0.0565 m (both hands) so the gripper base sits at wrist +x
0.1385 and the grasp/TCP fingertips reach ~0.242 m forward of wrist_yaw
(FT sensor -> TCP = 0.16 m) — matching the tcp_offset_x=0.242 used by the WBT
hybrid force controller + its mjswan viz. Symmetric left/right joint origins
(0 -+0.003 0.0565), comments updated to match.

Co-Authored-By: Claude Opus 4.8 (1M context) <noreply@anthropic.com>

File: src/holosoma/holosoma/data/robots/g1/g1_29dof_yam.urdf (robot description, URDF)
Before this commit: robot g1, 48 links, 47 joints
Joints:
- joint left_hand_palm_joint: origin xyz=0 -0.003 0.0295 rpy=0 -1.570796327 3.141592654 -> xyz=0 -0.003 0.0565 rpy=0 -1.570796327 3.141592654
- joint right_hand_palm_joint: origin xyz=0 0.003 0.0295 rpy=0 -1.570796327 3.141592654 -> xyz=0 0.003 0.0565 rpy=0 -1.570796327 3.141592654
